Commit message: today: sync with physical robot: success

File: src/gen3_description/description/kinova_gen3.urdf (robot description, URDF)
Before this commit: robot gen3_, 31 links, 30 joints
Links:
- link gen3_base_link: geometry collision mesh filename=package://gen3_description/meshes/gen3_arm_collision/base_l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; visual mesh filename=package://gen3_description/meshes/gen3_arm_visual/base_link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
- link gen3_bracelet_link: geometry collision mesh filename=package://gen3_description/meshes/gen3_arm_collision/bracel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; visual mesh filename=package://gen3_description/meshes/gen3_arm_visual/bracelet_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
- link gen3_forearm_link: geometry collision mesh filename=package://gen3_description/meshes/gen3_arm_collision/forear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; visual mesh filename=package://gen3_description/meshes/gen3_arm_visual/forearm_l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
- link gen3_half_arm_1_link: geometry collision mesh filename=package://gen3_description/meshes/gen3_arm_collision/half_a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; visual mesh filename=package://gen3_description/meshes/gen3_arm_visual/half_arm_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
- link gen3_half_arm_2_link: geometry collision mesh filename=package://gen3_description/meshes/gen3_arm_collision/half_a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; visual mesh filename=package://gen3_description/meshes/gen3_arm_visual/half_arm_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
- link gen3_robotiq_85_base_link: geometry collision mesh filename=package://gen3_description/meshes/g2f85_collision/robotiq_b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; visual mesh filename=package://gen3_description/meshes/g2f85_visual/robotiq_base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
- link gen3_robotiq_85_left_finger_link: geometry collision mesh filename=package://gen3_description/meshes/g2f85_collision/left_fing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; visual mesh filename=package://gen3_description/meshes/g2f85_visual/left_finger.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
- link gen3_robotiq_85_left_finger_tip_link: geometry collision mesh filename=package://gen3_description/meshes/g2f85_collision/left_fing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; visual mesh filename=package://gen3_description/meshes/g2f85_visual/left_finger_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
- link gen3_robotiq_85_left_inner_knuckle_link: geometry collision mesh filename=package://gen3_description/meshes/g2f85_collision/left_inne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; visual mesh filename=package://gen3_description/meshes/g2f85_visual/left_inner_k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
- link gen3_robotiq_85_left_knuckle_link: geometry collision mesh filename=package://gen3_description/meshes/g2f85_collision/left_knuc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; visual mesh filename=package://gen3_description/meshes/g2f85_visual/left_knuckle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
- link gen3_robotiq_85_right_finger_link: geometry collision mesh filename=package://gen3_description/meshes/g2f85_collision/right_fin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; visual mesh filename=package://gen3_description/meshes/g2f85_visual/right_finger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
- link gen3_robotiq_85_right_finger_tip_link: geometry collision mesh filename=package://gen3_description/meshes/g2f85_collision/right_fin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; visual mesh filename=package://gen3_description/meshes/g2f85_visual/right_finger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
- link gen3_robotiq_85_right_inner_knuckle_link: geometry collision mesh filename=package://gen3_description/meshes/g2f85_collision/right_inn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; visual mesh filename=package://gen3_description/meshes/g2f85_visual/right_inner_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
- link gen3_robotiq_85_right_knuckle_link: geometry collision mesh filename=package://gen3_description/meshes/g2f85_collision/right_knu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; visual mesh filename=package://gen3_description/meshes/g2f85_visual/right_knuckl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
- link gen3_shoulder_link: geometry collision mesh filename=package://gen3_description/meshes/gen3_arm_collision/should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; visual mesh filename=package://gen3_description/meshes/gen3_arm_visual/shoulder_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
- link gen3_spherical_wrist_1_link: geometry collision mesh filename=package://gen3_description/meshes/gen3_arm_collision/spheri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; visual mesh filename=package://gen3_description/meshes/gen3_arm_visual/spherical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
- link gen3_spherical_wrist_2_link: geometry collision mesh filename=package://gen3_description/meshes/gen3_arm_collision/spheri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; visual mesh filename=package://gen3_description/meshes/gen3_arm_visual/spherical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
- link wrist_camera_mount_link: geometry collision mesh filename=package://gen3_description/meshes//realsense_bracket_for_ki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; visual mesh filename=package://gen3_description/meshes/realsense_bracket_for_kin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

Commit message: changed robot urdf representations

File: src/gen3_description/description/kinova_gen3.urdf (robot description, URDF)
Before this commit: robot gen3_, 31 links, 30 joints
Joints:
- joint gen3_robotiq_85_left_inner_knuckle_joint: mimic joint=gen3_robotiq_85_left_knuckle_joint -> joint=gen3_robotiq_85_left_knuckle_joint multiplier=-1
- joint gen3_robotiq_85_right_finger_tip_joint: mimic joint=gen3_robotiq_85_left_knuckle_joint -> joint=gen3_robotiq_85_left_knuckle_joint multiplier=-1
