Commit message: modified structure

File: src/gen3_description/description/robotiq_2f85.urdf.xacro (robot description, xacro)
@@ -148,5 +148,5 @@
     <axis xyz="0 -1 0"/>
     <origin rpy="0 0 0" xyz="0.0127 0.0 0.06142"/>
-    <mimic joint="gen3_robotiq_85_left_knuckle_joint" multiplier="1"/>
+    <mimic joint="gen3_robotiq_85_left_knuckle_joint" />
   </joint>
   <joint name="gen3_robotiq_85_right_inner_knuckle_joint" type="continuous">
@@ -169,5 +169,5 @@
     <axis xyz="0 -1 0"/>
     <origin rpy="0 0 0" xyz="-0.0056 0.0 0.0471"/>
-    <mimic joint="gen3_robotiq_85_left_knuckle_joint" multiplier="1"/>
+    <mimic joint="gen3_robotiq_85_left_knuckle_joint" />
   </joint>
 </robot>
